File: Can_pHat_5.0.kicad_pcb (KiCad board)
At the start: 2 copper layers, 65 x 30 mm, 26 parts, among them J1 RaspberryPi40PinHeader, J2 DB9_Female, J3 Screw_Terminal_01x02, U2 MCP2515-EST, U3 MCP2551-I-SN, U4 24LC01, Y1 8MHz

Commit message: Changed IC combination (MCP2515, MCP2551) to a single IC (MCP25625). A smaller solution while maintaining the same cost (Or reducing it on larger volumes).
Parts:
- removed R6: 10k, Resistors_SMD:R_1206_HandSoldering
- removed R7: 22k, Resistors_SMD:R_1206_HandSoldering
- removed the REF** at (78.5, 43.5)
- removed the REF*** at (71.4, 27.2)
- removed U2: MCP2515-EST, Housings_SOIC:SOIC-18W_7.5x11.6mm_Pitch1.27mm
- removed U3: MCP2551-I-SN, Housings_SOIC:SOIC-8_3.9x4.9mm_Pitch1.27mm
- added C6: 0.1uF, Capacitors_SMD:C_1206_HandSoldering, F.Cu at (21.7, 29.8)
- added U1: MCP25625-x-SS, Housings_SSOP:SSOP-28_5.3x10.2mm_Pitch0.65mm, F.Cu at (31.1, 31.1)
- C1, C2: value 820pF -> 0.1uF
- moved C3 22.1 mm to (27.3, 38.1), turned to 180 degrees
- moved C1 15.8 mm to (21.7, 34.9), turned to 180 degrees
- moved C4 14.5 mm to (34.2, 38.1)
- moved Y1 12.5 mm to (33.5, 43.2)
- moved C2 9.93 mm to (21.7, 32.4), turned to 180 degrees
- moved R1 2.22 mm to (40.7, 27.9)
Connections:
- C1 pad 1: GND -> +3V3
- C1 pad 2: +5V -> GND
- J1 pad 10: Net-(J1-Pad10) -> (no net)
- J1 pad 11: Net-(J1-Pad11) -> (no net)
- J1 pad 12: Net-(J1-Pad12) -> (no net)
- J1 pad 13: Net-(J1-Pad13) -> (no net)
- J1 pad 15: Net-(J1-Pad15) -> (no net)
- J1 pad 16: Net-(J1-Pad16) -> (no net)
- J1 pad 18: Net-(J1-Pad18) -> (no net)
- J1 pad 22: Net-(J1-Pad22) -> (no net)
- J1 pad 26: Net-(J1-Pad26) -> (no net)
- J1 pad 3: Net-(J1-Pad3) -> (no net)
- J1 pad 30: Net-(J1-Pad30) -> (no net)
- J1 pad 31: Net-(J1-Pad31) -> (no net)
- J1 pad 32: Net-(J1-Pad32) -> (no net)
- J1 pad 33: Net-(J1-Pad33) -> (no net)
- J1 pad 35: Net-(J1-Pad35) -> (no net)
- J1 pad 36: Net-(J1-Pad36) -> (no net)
- J1 pad 37: Net-(J1-Pad37) -> (no net)
- J1 pad 38: Net-(J1-Pad38) -> (no net)
- J1 pad 40: Net-(J1-Pad40) -> (no net)
- J1 pad 5: Net-(J1-Pad5) -> (no net)
- J1 pad 7: Net-(J1-Pad7) -> (no net)
- J1 pad 8: Net-(J1-Pad8) -> (no net)
- J2 pad 1: Net-(J2-Pad1) -> (no net)
- J2 pad 5: Net-(J2-Pad5) -> (no net)
- J2 pad 8: Net-(J2-Pad8) -> (no net)
- J2 pad 9: +12V -> (no net)
Routing:
- net Net-(R6-Pad2): track 17.8 -> 0.00 mm
- net Net-(R1-Pad2): track 23.2 -> 7.09 mm, vias 2 -> 0
- net CAN+: track 63.8 -> 78.1 mm
- net CAN-: track 65.1 -> 78.1 mm
- net OSC2: track 22.4 -> 9.77 mm
- net Net-(R6-Pad1): track 12.2 -> 0.00 mm, vias 2 -> 0
- net ~CS: track 35.4 -> 24.0 mm
- net Net-(U2-Pad1): track 11.3 -> 0.00 mm
- net SO: track 30.3 -> 19.1 mm, vias 1 -> 0
- net SI: track 25.8 -> 15.3 mm, vias 0 -> 1
- net OSC1: track 19.6 -> 9.15 mm
- net Net-(U1-Pad21): track 0.00 -> 8.87 mm, vias 0 -> 2
- net +5V: track 53.6 -> 46.5 mm
- net GND: track 20.0 -> 25.5 mm, vias 8 -> 7
- net Net-(U1-Pad20): track 0.00 -> 4.91 mm
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Other:
- board text added: "Rev 1.2"
